File: Hardware/Master/Repositor Automático V8 (Primer Final)/Repositor Automático V8 (Primer Final).kicad_sch (KiCad schematic)
At the start: 53 parts, among them IC1 TB67H450AFNG,EL, IC2 TB67H450AFNG,EL, IC3 TB67H450AFNG,EL, IC4 MP2307, J1 Alimentacion 12V, J1 Screw_Terminal_01x10, J11 Final de carrera, J2 UART, J3 Motor2, J4 Motor1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

Commit message: Corrección de errores
Se agrego un Led de prueba para testear el funcionamiento del Esp32 WROOM y se corrigió la resistencia pull-up del pin BOOT
Parts:
- removed C8: 0.1u, Capacitor_SMD:C_1206_3216Metric, symbol Device:C
- removed R16, R17: 100k, Resistor_SMD:R_1206_3216Metric, symbol Device:R
- removed SWJ2: SW_MEC_5G, Button_Switch_SMD:SW_Push_SPST_NO_Alps_SKRK, symbol Switch:SW_MEC_5G
- added C23, C24: 0.1u, Capacitor_SMD:C_1206_3216Metric, symbol Device:C
- added D2: LED, LED_SMD:LED_1206_3216Metric, symbol Device:LED
- added R8: 330, Resistor_SMD:R_1206_3216Metric, symbol Device:R
- added R9: 4.7k, Resistor_SMD:R_1206_3216Metric, symbol Device:R
- added SWJ3: SW_MEC_5G, Button_Switch_SMD:SW_Push_SPST_NO_Alps_SKRK, symbol Switch:SW_MEC_5G
- R18: value 10k -> 4.7k
Connections:
- net 3V3: now also R9.2
- net BOOT: now also C23.2, C24.2, R9.1, SWJ3.2 (B)
- net EN: now also C7.2, SWJ1.2 (B)
- net GND: now also C23.1, C24.1, D2.1 (K), SWJ3.1 (A)
- net Led prueba: now reaches U10.24 (IO2)
- net Led prueba: now also R8.1
- new net: D2.2 (A), R8.2
- no-connect marks 13 -> 12
Other:
- note added: "Led de prueba"
- moved on the sheet: C17, C7, C9, J1, R18, SWJ1

Commit message: Diseño final con correccion de Errores
Connections:
- net 3V3: now also R4.1
- net FC: now also C17.2, J11.1 (Pin_1), R4.2; no longer R4.1
Changed lines of the file:
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@@
     (effects (font (size 1.27 1.27)) (justify left bottom))
   )
-  (label "FC" (at 56.515 111.76 0) (fields_autoplaced)
+  (label "FC" (at 80.645 111.76 0) (fields_autoplaced)
     (effects (font (size 1.27 1.27)) (justify left bottom))
   )
@@
     (effects (font (size 1.27 1.27)) (justify left bottom))
   )
+  (label "3V3" (at 56.515 111.76 0) (fields_autoplaced)
+    (effects (font (size 1.27 1.27)) (justify left bottom))
+  )

Commit message: Correccion de errores diseño final
Connections:
- net 3V3: no longer R4.1
- net FC: now also R4.1; no longer C17.2, J11.1 (Pin_1), R4.2
- new net: C17.2, J11.1 (Pin_1), R4.2
Changed lines of the file:
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@@
     (effects (font (size 1.27 1.27)) (justify left bottom))
   )
-  (label "FC" (at 80.645 111.76 0) (fields_autoplaced)
+  (label "FC" (at 56.515 111.76 0) (fields_autoplaced)
     (effects (font (size 1.27 1.27)) (justify left bottom))
   )
@@
     (effects (font (size 1.27 1.27)) (justify left bottom))
   )
-  (label "3V3" (at 56.515 111.76 0) (fields_autoplaced)
-    (effects (font (size 1.27 1.27)) (justify left bottom))
-  )
